File: PnP_Power/PnP_Power.kicad_pcb (KiCad board)
At the start: 2 copper layers, 120.7 x 121.2 mm, 89 parts, among them J1 Barrel Jack 5mm x 2.5mm 54-00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, J2 Conn_02x03_Odd_Even, J3 Conn_02x03_Odd_Even, J4 Conn_02x03_Odd_Even, J5 Conn_02x03_Odd_Even, J6 Conn_02x03_Odd_Even, J7 Conn_02x03_Odd_Even, J8 Conn_01x03_Pin, J9 Conn_01x03_Pin, Q1 PMOS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

Commit message: Fix DRC issues
Routing:
- net +5V: track 514.8 -> 537.7 mm
- net GND: vias 420 -> 352
