File: PnP_Power/PnP_Power.kicad_pcb (KiCad board)
At the start: 2 copper layers, 120.7 x 121.2 mm, 89 parts, among them J1 Barrel Jack 5mm x 2.5mm 54-00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, J2 Conn_02x03_Odd_Even, J3 Conn_02x03_Odd_Even, J4 Conn_02x03_Odd_Even, J5 Conn_02x03_Odd_Even, J6 Conn_02x03_Odd_Even, J7 Conn_02x03_Odd_Even, J8 Conn_01x03_Pin, J9 Conn_01x03_Pin, Q1 PMOS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

Commit message: Final board trust me
Parts:
- moved H3 0.92 mm to (108.2, 169.2)
- moved H4 0.76 mm to (223.3, 169.2)
- moved H1 0.51 mm to (108.2, 52.3)
Routing:
- net +12V: track 296.1 -> 297.0 mm
Other:
- board size 120.7 x 121.2 mm -> 121.2 x 122.9 mm
